File: hardware/ENTRENADORA2.kicad_pcb (KiCad board)
At the start: 2 copper layers, 102 x 54 mm, 0 parts

Commit message: co
Parts:
- added C1: C, Capacitor_SMD:C_0805_2012Metric_Pad1.15x1.40mm_HandSolder, F.Cu at (139.3, 110.7)
- added C2: C, Capacitor_SMD:C_0805_2012Metric_Pad1.15x1.40mm_HandSolder, F.Cu at (163.0, 83.7)
- added C3: C, Capacitor_SMD:C_0805_2012Metric_Pad1.15x1.40mm_HandSolder, F.Cu at (148.9, 101.3)
- added C4: C, Capacitor_SMD:C_0805_2012Metric_Pad1.15x1.40mm_HandSolder, F.Cu at (144.1, 103.0)
- added C5: C, Capacitor_SMD:C_0805_2012Metric_Pad1.15x1.40mm_HandSolder, F.Cu at (153.6, 101.5)
- added C6: C, Capacitor_SMD:C_0805_2012Metric_Pad1.15x1.40mm_HandSolder, F.Cu at (148.8, 107.2)
- added C7: C, Capacitor_SMD:C_0805_2012Metric_Pad1.15x1.40mm_HandSolder, F.Cu at (180.9, 75.5)
- added D1: D_Schottky, Diode_SMD:D_SOD-123, F.Cu at (139.6, 92.5)
- added D10: LED_Small, LED_SMD:LED_0805_2012Metric_Pad1.15x1.40mm_HandSolder, F.Cu at (134.5, 101.7)
- added D11: LED_Small, LED_SMD:LED_0805_2012Metric_Pad1.15x1.40mm_HandSolder, F.Cu at (134.5, 104.8)
- added D12: LED_Small, LED_SMD:LED_0805_2012Metric_Pad1.15x1.40mm_HandSolder, F.Cu at (139.3, 104.8)
- added D13: LED_Small, LED_SMD:LED_0805_2012Metric_Pad1.15x1.40mm_HandSolder, F.Cu at (144.1, 100.0)
- added D14: LED_Small, LED_SMD:LED_0805_2012Metric_Pad1.15x1.40mm_HandSolder, F.Cu at (166.7, 79.7)
- added D15: LED_Small, LED_SMD:LED_0805_2012Metric_Pad1.15x1.40mm_HandSolder, F.Cu at (158.2, 86.7)
- added D16: LED_Small, LED_SMD:LED_0805_2012Metric_Pad1.15x1.40mm_HandSolder, F.Cu at (158.2, 83.7)
- added D17: LED_Small, LED_SMD:LED_0805_2012Metric_Pad1.15x1.40mm_HandSolder, F.Cu at (134.5, 110.9)
- added D18: LED, LED_SMD:LED_0805_2012Metric_Pad1.15x1.40mm_HandSolder, F.Cu at (134.5, 107.8)
- added D2: LED_Small, LED_SMD:LED_0805_2012Metric_Pad1.15x1.40mm_HandSolder, F.Cu at (149.8, 95.4)
- added D3: LED_Small, LED_SMD:LED_0805_2012Metric_Pad1.15x1.40mm_HandSolder, F.Cu at (176.2, 69.6)
- added D4: LED_Small, LED_SMD:LED_0805_2012Metric_Pad1.15x1.40mm_HandSolder, F.Cu at (139.2, 95.7)
- added D5: LED_Small, LED_SMD:LED_0805_2012Metric_Pad1.15x1.40mm_HandSolder, F.Cu at (139.3, 101.7)
- added D6: LED_Small, LED_SMD:LED_0805_2012Metric_Pad1.15x1.40mm_HandSolder, F.Cu at (149.8, 92.3)
- added D7: LED_Small, LED_SMD:LED_0805_2012Metric_Pad1.15x1.40mm_HandSolder, F.Cu at (139.2, 98.7)
- added D8: LED_Small, LED_SMD:LED_0805_2012Metric_Pad1.15x1.40mm_HandSolder, F.Cu at (166.7, 76.7)
- added D9: LED_Small, LED_SMD:LED_0805_2012Metric_Pad1.15x1.40mm_HandSolder, F.Cu at (144.0, 97.0)
- added F1: Polyfuse_Small, Fuse:Fuse_0805_2012Metric_Pad1.15x1.40mm_HandSolder, F.Cu at (163.0, 86.6)
- added J1: , Connector_PinHeader_2.54mm:PinHeader_2x02_P2.54mm_Vertical, F.Cu at (139.1, 85.9)
- added J2: Conn_01x02, Connector_PinHeader_2.54mm:PinHeader_1x02_P2.54mm_Vertical, F.Cu at (134.4, 93.1)
- added J3: USB_B_Micro, Connectors_EC:629105150521, F.Cu at (149.9, 70.8)
- added J4: , Connector_PinHeader_2.54mm:PinHeader_1x01_P2.54mm_Vertical, F.Cu at (139.2, 117.5)
- added J5: , Connector_PinHeader_2.54mm:PinHeader_1x01_P2.54mm_Vertical, F.Cu at (144.0, 112.7)
- added J6: , Connector_PinHeader_2.54mm:PinHeader_2x02_P2.54mm_Vertical, F.Cu at (150.9, 85.9)
- added J7: Conn_01x02, Connector_PinHeader_2.54mm:PinHeader_1x02_P2.54mm_Vertical, F.Cu at (134.4, 85.9)
- added J8: , Connector_PinHeader_2.54mm:PinHeader_1x02_P2.54mm_Vertical, F.Cu at (146.3, 85.9)
- added J9: , Connector_PinHeader_2.54mm:PinHeader_1x01_P2.54mm_Vertical, F.Cu at (158.3, 99.4)
- added R1: R_Small, Resistor_SMD:R_0805_2012Metric_Pad1.15x1.40mm_HandSolder, F.Cu at (148.8, 104.2)
- added R10: R, Resistor_SMD:R_0805_2012Metric_Pad1.15x1.40mm_HandSolder, F.Cu at (180.9, 72.6)
- added R11: R, Resistor_SMD:R_0805_2012Metric_Pad1.15x1.40mm_HandSolder, F.Cu at (181.0, 69.6)
- added R12: R, Resistor_SMD:R_0805_2012Metric_Pad1.15x1.40mm_HandSolder, F.Cu at (171.4, 76.6)
- added R13: R_Small, Resistor_SMD:R_0805_2012Metric_Pad1.15x1.40mm_HandSolder, F.Cu at (144.1, 105.9)
- added R14: R_Small, Resistor_SMD:R_0805_2012Metric_Pad1.15x1.40mm_HandSolder, F.Cu at (154.5, 92.7)
- added R15: R_Small, Resistor_SMD:R_0805_2012Metric_Pad1.15x1.40mm_HandSolder, F.Cu at (171.4, 79.6)
- added R16: R_Small, Resistor_SMD:R_0805_2012Metric_Pad1.15x1.40mm_HandSolder, F.Cu at (154.5, 95.6)
- added R17: R_Small, Resistor_SMD:R_0805_2012Metric_Pad1.15x1.40mm_HandSolder, F.Cu at (176.2, 76.6)
- added R18: R_Small, Resistor_SMD:R_0805_2012Metric_Pad1.15x1.40mm_HandSolder, F.Cu at (159.3, 92.7)
- added R19: R_Small, Resistor_SMD:R_0805_2012Metric_Pad1.15x1.40mm_HandSolder, F.Cu at (148.9, 98.3)
- added R2: R_Small, Resistor_SMD:R_0805_2012Metric_Pad1.15x1.40mm_HandSolder, F.Cu at (163.0, 89.6)
- added R20: R_Small, Resistor_SMD:R_0805_2012Metric_Pad1.15x1.40mm_HandSolder, F.Cu at (167.7, 82.7)
- added R21: R, Resistor_SMD:R_0805_2012Metric_Pad1.15x1.40mm_HandSolder, F.Cu at (134.5, 116.8)
- added R22: R, Resistor_SMD:R_0805_2012Metric_Pad1.15x1.40mm_HandSolder, F.Cu at (158.2, 89.7)
- added R23: R, Resistor_SMD:R_0805_2012Metric_Pad1.15x1.40mm_HandSolder, F.Cu at (167.7, 85.6)
- added R24: R, Resistor_SMD:R_0805_2012Metric_Pad1.15x1.40mm_HandSolder, F.Cu at (153.6, 98.6)
- added R25: R, Resistor_SMD:R_0805_2012Metric_Pad1.15x1.40mm_HandSolder, F.Cu at (144.0, 108.9)
- added R26: R, Resistor_SMD:R_0805_2012Metric_Pad1.15x1.40mm_HandSolder, F.Cu at (139.3, 113.7)
- added R27: R, Resistor_SMD:R_0805_2012Metric_Pad1.15x1.40mm_HandSolder, F.Cu at (185.7, 69.6)
- added R3: R_Small, Resistor_SMD:R_0805_2012Metric_Pad1.15x1.40mm_HandSolder, F.Cu at (172.5, 82.5)
- added R4: R_Small, Resistor_SMD:R_0805_2012Metric_Pad1.15x1.40mm_HandSolder, F.Cu at (134.5, 119.8)
- added R5: R_Small, Resistor_SMD:R_0805_2012Metric_Pad1.15x1.40mm_HandSolder, F.Cu at (159.3, 95.6)
- added R6: R_Small, Resistor_SMD:R_0805_2012Metric_Pad1.15x1.40mm_HandSolder, F.Cu at (176.2, 79.6)
- added R7: R_Small, Resistor_SMD:R_0805_2012Metric_Pad1.15x1.40mm_HandSolder, F.Cu at (139.3, 107.8)
- added R8: R_Small, Resistor_SMD:R_0805_2012Metric_Pad1.15x1.40mm_HandSolder, F.Cu at (176.2, 72.6)
- added R9: R, Resistor_SMD:R_0805_2012Metric_Pad1.15x1.40mm_HandSolder, F.Cu at (134.5, 113.9)
- added SW1: , Button_Switch_SMD:SW_SPST_TL3342, F.Cu at (159.5, 71.6)
- added SW2: , Button_Switch_SMD:SW_SPST_TL3342, F.Cu at (146.4, 80.1)
- added SW3: , Button_Switch_SMD:SW_SPST_TL3342, F.Cu at (185.0, 86.9)
- added SW4: , Button_Switch_SMD:SW_SPST_TL3342, F.Cu at (136.9, 80.1)
- added SW5: , Button_Switch_SMD:SW_SPST_TL3342, F.Cu at (185.0, 94.0)
- added SW6: , Button_Switch_SMD:SW_SPST_TL3342, F.Cu at (169.0, 71.6)
- added SW7: , Button_Switch_SMD:SW_SPST_TL3342, F.Cu at (159.5, 78.7)
- added SW8: , Button_Switch_SMD:SW_SPST_TL3342, F.Cu at (194.6, 86.9)
- added SW9: , Button_Switch_SMD:SW_SPST_TL3342, F.Cu at (194.6, 94.0)
- added U1: AP2112K-3.3TRG1, Package_TO_SOT_SMD:SOT-23-5, F.Cu at (170.6, 93.0)
- added U2: MCP73831-2-OT, Package_TO_SOT_SMD:SOT-23-5, F.Cu at (144.9, 93.1)
- added U3: PIC18F4550-IP, Package_DIP:DIP-40_W15.24mm, F.Cu at (115.3, 70.2)
- added Y1: Crystal, Crystal:Crystal_HC49-U_Vertical, F.Cu at (136.1, 71.4)
Other:
- board size 102 x 54 mm -> 100 x 54 mm
